Commit message: Adjeusted xacro fule parameters

File: src/erp42_description/urdf/erp42_model.xacro (robot description, xacro)
@@ -8,8 +8,4 @@
         <!-- Constants -->
         <xacro:property name="PI" value="3.14159"/>
-        <!-- Base dimensions -->
-        <xacro:property name="base_x_size" value="2.020" />
-        <xacro:property name="base_y_size" value="1.160" />
-        <xacro:property name="base_z_size" value="0.550" />
         <!-- Wheel geometry (from 175/60R13) -->
         <xacro:property name="wheel_length" value="0.175" />
@@ -35,4 +31,17 @@
                 <inertia ixx="20.43" ixy="0.584" ixz="-0.191" iyy="54.197" iyz="-0.2449" izz="72.2588"/>
             </inertial>
+            <!-- Chassis -->
+            <collision>
+                <origin xyz="0.02 0 0" rpy="0 0 0" />
+                <geometry>
+                    <box size="1.580 0.950 0.316"/>
+                </geometry>
+            </collision>
+            <visual>
+                <origin xyz="0 0 0" rpy="0 0 0" />
+                <geometry>
+                    <mesh filename="file://$(find erp42_description)/meshes/erp42_chassis.dae"  scale="0.001 0.001 0.001"/>
+                </geometry>
+            </visual>
             <!-- Front bumper -->
             <collision>
@@ -59,11 +68,4 @@
                 <geometry>
                     <mesh filename="file://$(find erp42_description)/meshes/erp42_bumper.dae"  scale="0.001 0.001 0.001"/>
-                </geometry>
-            </visual>
-            <!-- Chassis -->
-            <visual>
-                <origin xyz="0 0 0" rpy="0 0 0" />
-                <geometry>
-                    <mesh filename="file://$(find erp42_description)/meshes/erp42_chassis.dae"  scale="0.001 0.001 0.001"/>
                 </geometry>
             </visual>

Commit message: chassis link merged into base_link

File: src/erp42_description/urdf/erp42_model.xacro (robot description, xacro)
@@ -22,7 +22,5 @@
         <link name="base_footprint"/>
         <!-- Base link -->
-        <link name="base_link"/>
-        <!-- Chassis -->
-        <link name="chassis">
+        <link name="base_link">
             <!-- Inertia -->
             <inertial>
@@ -100,10 +98,4 @@
             <child link="base_link" />
         </joint>
-        <!-- base_link to chassis -->
-        <joint name="chassis_joint" type="fixed">
-            <origin xyz="0 0 0" rpy="0 0 0" />
-            <parent link="base_link" />
-            <child link="chassis" />
-        </joint>
         <!-- base_link to front_left_steering_hub -->
         <joint name="front_left_steering_hub_joint" type="revolute">
