Commit message: Update joint velocity limit in rear wheel xacro

File: src/erp42_gazebo_sim/urdf/erp42_rear_wheel.xacro (robot description, xacro)
@@ -53,5 +53,5 @@
             <axis xyz = "0 1 0"/>
             <!-- Limits -->
-            <limit effort = "1000000.0" velocity = "${7.0 / radius}"/>
+            <limit effort = "1000000.0" velocity = "${10.0 / radius}"/>
         </joint>
         <!-- Friction settings -->
