Commit message: Vehicle parameter updated

File: src/erp42_gazebo_sim/urdf/erp42_front_wheel.xacro (robot description, xacro)
@@ -87,6 +87,6 @@
                 lower    = "${-1.2 * radians(25)}"
                 upper    = "${ 1.2 * radians(25)}"
-                effort   = "1000"
-                velocity = "1.0"
+                velocity = "${radians(25)}"
+                effort   = "1000000.0"
             />
         </joint>
@@ -101,5 +101,5 @@
             <axis xyz = "0 1 0"/>
             <!-- Limits -->
-            <limit effort = "10000.0" velocity = "${7.0 / radius}"/>
+            <limit effort = "1000000.0" velocity = "${7.0 / radius}"/>
         </joint>
         <!-- Friction settings -->

Commit message: Vehicle parameter edited

File: src/erp42_gazebo_sim/urdf/erp42_front_wheel.xacro (robot description, xacro)
@@ -87,5 +87,5 @@
                 lower    = "${-1.2 * radians(25)}"
                 upper    = "${ 1.2 * radians(25)}"
-                velocity = "${radians(25)}"
+                velocity = "${ 2.0 * radians(25)}"
                 effort   = "1000000.0"
             />
@@ -101,5 +101,5 @@
             <axis xyz = "0 1 0"/>
             <!-- Limits -->
-            <limit effort = "1000000.0" velocity = "${7.0 / radius}"/>
+            <limit effort = "1000000.0" velocity = "${10.0 / radius}"/>
         </joint>
         <!-- Friction settings -->

Commit message: Vehicle parameter edited

File: src/erp42_gazebo_sim/urdf/erp42_front_wheel.xacro (robot description, xacro)
@@ -82,10 +82,10 @@
             <axis xyz = "0 0 1"/>
             <!-- Dynamics -->
-            <dynamics friction = "10.0" damping = "1.0"/>
+            <dynamics friction = "0.1" damping = "0.1"/>
             <!-- Limits -->
             <limit
                 lower    = "${-1.2 * radians(25)}"
                 upper    = "${ 1.2 * radians(25)}"
-                velocity = "${radians(25)}"
+                velocity = "${ 2.0 * radians(25)}"
                 effort   = "1000000.0"
             />
@@ -101,5 +101,5 @@
             <axis xyz = "0 1 0"/>
             <!-- Limits -->
-            <limit effort = "1000000.0" velocity = "${7.0 / radius}"/>
+            <limit effort = "1000000.0" velocity = "${10.0 / radius}"/>
         </joint>
         <!-- Friction settings -->

Commit message: Vehicle parameter edited

File: src/erp42_gazebo_sim/urdf/erp42_front_wheel.xacro (robot description, xacro)
@@ -13,5 +13,5 @@
         <xacro:property name  = "izz" value = "${1/2  * mass * radius * radius}"/>
         <!-- Steer properties -->
-        <xacro:property name = "dummy_mass"   value = "5"  />
+        <xacro:property name = "dummy_mass"   value = "1"  />
         <xacro:property name = "dummy_radius" value = "0.1"/>
         <xacro:property name = "dummy_ixx" value = "${3/5 * dummy_mass * dummy_radius * dummy_radius}"/>
@@ -87,5 +87,5 @@
                 lower    = "${-1.2 * radians(25)}"
                 upper    = "${ 1.2 * radians(25)}"
-                velocity = "${ 2.0 * radians(25)}"
+                velocity = "${ 4.0 * radians(25)}"
                 effort   = "1000000.0"
             />
@@ -101,5 +101,5 @@
             <axis xyz = "0 1 0"/>
             <!-- Limits -->
-            <limit effort = "1000000.0" velocity = "${10.0 / radius}"/>
+            <limit effort = "360.0" velocity = "${7.0 / radius}"/>
         </joint>
         <!-- Friction settings -->
